File: hw/Asius1/Asius1.kicad_pcb (KiCad board)
At the start: 4 copper layers, 40 x 60 mm, 48 parts, among them J1 SPI1, J2 Extra, J3 PWR, SW1 DFU, SW2 RESET, U1 STM32F413RGT6, U2 SN65HVD230DR, U3 SN65HVD230DR, U4 SN65HVD230DR, U5 AMS1117-3.3, U6 SN65HVD230DR, Y2 Crystal_GND24

Commit message: Asius2 kicad
Parts:
- USBC1: value OBD-C -> ~
Connections:
- USBC1 pad 0: GND -> (no net)
