File: hw/Asius1/Asius1.kicad_sch (KiCad schematic)
At the start: 48 parts, among them J1 SPI1, J2 Extra, J3 PWR, SW1 DFU, SW2 RESET, U1 STM32F413RGT6, U2 SN65HVD230DR, U3 SN65HVD230DR, U4 SN65HVD230DR, U5 AMS1117-3.3, U6 SN65HVD230DR, Y2 Crystal_GND24

Commit message: Asius2 kicad
Parts:
- USBC1: value OBD-C -> ~; MPN TYPE-C-31-M-04 -> (none); Manufacturer Korean Hroparts Elec -> 韩国韩荣; Manufacturer Part (none) -> TYPE-C-31-M-04
Connections:
- net GND: now also USBC1.S1 (0), USBC1.S2 (0), USBC1.S3 (0), USBC1.S4 (0); no longer USBC1.0
Changed lines of the file:
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@@
 	)
 	(junction
+		(at 57.15 118.11)
+		(diameter 0)
+		(color 0 0 0 0)
+	)
+	(junction
 		(at 222.25 133.35)
 		(diameter 0)
@@
 		(color 0 0 0 0)
 	)
-	(junction
-		(at 57.15 118.11)
-		(diameter 0)
-		(color 0 0 0 0)
-	)
 	(no_connect
 		(at 196.85 72.39)
@@
 	)
 	(symbol
+		(lib_id "1_my_custom_symbol_lib:TYPE-C-31-M-04")
+		(at 43.18 104.14 0)
+		(unit 1)
+		(exclude_from_sim no)
+		(in_bom yes)
+		(on_board yes)
+		(dnp no)
+		(fields_autoplaced yes)
+		(property "Reference" "USBC1"
+			(at 46.5933 82.55 0)
+			(effects
+				(font
+					(size 1.27 1.27)
+				)
+				(justify left)
+			)
+		)
+		(property "Value" "~"
+			(at 46.5933 85.09 0)
+			(effects
+				(font
+					(size 1.27 1.27)
+				)
+				(justify left)
+			)
+		)
+		(property "Footprint" "1_My_custom_library:USB-C-SMD_TYPE-C-USB-20"
+			(at 43.18 104.14 0)
+			(effects
+				(font
+					(size 1.27 1.27)
+				)
+				(hide yes)
+			)
+		)
+		(property "Datasheet" "https://item.szlcsc.com/datasheet/TYPE-C-31-M-04/140304.html"
+			(at 43.18 104.14 0)
+			(effects
+				(font
+					(size 1.27 1.27)
+				)
+				(hide yes)
+			)
+		)
+		(property "Description" "Connector Type:Type-C Protocol Standard:- Gender:Female Number of Contacts:24P Number of Ports:1"
+			(at 43.18 104.14 0)
+			(effects
+				(font
+					(size 1.27 1.27)
+				)
+				(hide yes)
+			)
+		)
+		(property "Manufacturer Part" "TYPE-C-31-M-04"
+			(at 43.18 104.14 0)
+			(effects
+				(font
+					(size 1.27 1.27)
+				)
+				(hide yes)
+			)
+		)
+		(property "Manufacturer" "韩国韩荣"
+			(at 43.18 104.14 0)
+			(effects
+				(font
+					(size 1.27 1.27)
+				)
+				(hide yes)
+			)
+		)
+		(property "Supplier Part" "C129018"
+			(at 43.18 104.14 0)
+			(effects
+				(font
+					(size 1.27 1.27)
+				)
+				(hide yes)
+			)
+		)
+		(property "Supplier" "LCSC"
+			(at 43.18 104.14 0)
+			(effects
+				(font
+					(size 1.27 1.27)
+				)
+				(hide yes)
+			)
+		)
+		(property "LCSC Part Name" "Type-C 母"
+			(at 43.18 104.14 0)
+			(effects
+				(font
+					(size 1.27 1.27)
+				)
+				(hide yes)
+			)
+		)
+		(pin "B4"
+		)
+		(pin "B5"
+		)
+		(pin "B6"
+		)
+		(pin "B7"
+		)
+		(pin "A7"
+		)
+		(pin "A6"
+		)
+		(pin "A5"
+		)
+		(pin "A4"
+		)
+		(pin "A3"
+		)
+		(pin "A2"
+		)
+		(pin "A1"
+		)
+		(pin "B12"
+		)
+		(pin "S1"
+		)
+		(pin "B10"
+		)
+		(pin "B11"
+		)
+		(pin "B1"
+		)
+		(pin "B2"
+		)
+		(pin "B3"
+		)
+		(pin "S4"
+		)
+		(pin "S3"
+		)
+		(pin "S2"
+		)
+		(pin "A12"
+		)
+		(pin "A11"
+		)
+		(pin "A10"
+		)
+		(pin "A9"
+		)
+		(pin "A8"
+		)
+		(pin "B8"
+		)
+		(pin "B9"
+		)
+		(instances
+			(project ""
+				(path "/c427f881-4211-43b6-9155-a5bf29a59f45"
+					(reference "USBC1")
+					(unit 1)
+				)
+			)
+		)
+	)
+	(symbol
 		(lib_id "MCU_ST_STM32F4:STM32F413RGTx")
 		(at 217.17 85.09 180)
@@
 					(unit 1)
 				)
-			)
-		)
-	)
-	(symbol
-		(lib_id "1_my_custom_symbol_lib:TYPE-C-31-M-04")
-		(at 43.18 104.14 0)
-		(unit 1)
-		(exclude_from_sim no)
-		(in_bom yes)
-		(on_board yes)
-		(dnp no)
-		(fields_autoplaced yes)
-		(property "Reference" "USBC1"
-			(at 46.5933 82.55 0)
-			(effects
-				(font
-					(size 1.27 1.27)
-				)
-				(justify left)
-				(hide yes)
-			)
-		)
-		(property "Value" "OBD-C"
-			(at 46.5933 85.09 0)
-			(effects
-				(font
-					(size 1.27 1.27)
-				)
-				(justify left)
-			)
-		)
-		(property "Footprint" "1_My_custom_library:USB-C-SMD_TYPE-C-USB-20"
-			(at 43.18 104.14 0)
-			(effects
-				(font
-					(size 1.27 1.27)
-				)
-				(hide yes)
-			)
-		)
-		(property "Datasheet" "https://item.szlcsc.com/datasheet/TYPE-C-31-M-04/140304.html"
-			(at 43.18 104.14 0)
-			(effects
-				(font
-					(size 1.27 1.27)
-				)
-				(hide yes)
-			)
-		)
-		(property "Description" "Connector Type:Type-C Protocol Standard:- Gender:Female Number of Contacts:24P Number of Ports:1"
-			(at 43.18 104.14 0)
-			(effects
-				(font
-					(size 1.27 1.27)
-				)
-				(hide yes)
-			)
-		)
-		(property "MPN" "TYPE-C-31-M-04"
-			(at 43.18 104.14 0)
-			(effects
-				(font
-					(size 1.27 1.27)
-				)
-				(hide yes)
-			)
-		)
-		(property "Manufacturer" "Korean Hroparts Elec"
-			(at 43.18 104.14 0)
-			(effects
-				(font
-					(size 1.27 1.27)
-				)
-				(hide yes)
-			)
-		)
-		(property "Supplier Part" "C129018"
-			(at 43.18 104.14 0)
-			(effects
-				(font
-					(size 1.27 1.27)
-				)
-				(hide yes)
-			)
-		)
-		(property "Supplier" "LCSC"
-			(at 43.18 104.14 0)
-			(effects
-				(font
-					(size 1.27 1.27)
-				)
-				(hide yes)
-			)
-		)
-		(property "LCSC Part Name" "Type-C 母"
-			(at 43.18 104.14 0)
-			(effects
-				(font
-					(size 1.27 1.27)
-				)
-				(hide yes)
-			)
-		)
-		(pin "A5"
-		)
-		(pin "B6"
-		)
-		(pin "0"
-		)
-		(pin "B3"
-		)
-		(pin "B9"
-		)
-		(pin "B11"
-		)
-		(pin "B7"
-		)
-		(pin "B4"
-		)
-		(pin "B12"
-		)
-		(pin "B5"
-		)
-		(pin "B8"
-		)
-		(pin "B10"
-		)
-		(pin "0"
-		)
-		(pin "B1"
-		)
-		(pin "B2"
-		)
-		(pin "A7"
-		)
-		(pin "A3"
-		)
-		(pin "A12"
-		)
-		(pin "A9"
-		)
-		(pin "A2"
-		)
-		(pin "A4"
-		)
-		(pin "A6"
-		)
-		(pin "A11"
-		)
-		(pin "A10"
-		)
-		(pin "A1"
-		)
-		(pin "0"
-		)
-		(pin "A8"
-		)
-		(pin "0"
-		)
-		(instances
-			(project ""
-				(path "/c427f881-4211-43b6-9155-a5bf29a59f45"
-					(reference "USBC1")
-					(unit 1)
-				)
