File: hw/Asius2/Asius2.kicad_pcb (KiCad board)
At the start: 6 copper layers, 40 x 60 mm, 77 parts, among them J1 PWR, J2 Hat, J3 Others, J4 Fan, J5 Audio, J6 SWD, SW1 DFU, SW2 RESET, U1 AMS1117-3.3, U2 TJA1042T, U3 TJA1042T, U4 TJA1042T, U5 TJA1042T, U6 LSM6DSOXTR, U7 STM32H725AGIx, Y1 Crystal_GND24

Commit message: v2
Parts:
- removed JP1: ~, Jumper:SolderJumper-2_P1.3mm_Bridged_RoundedPad1.0x1.5mm
- added C42: 3.3nF, Capacitor_SMD:C_0603_1608Metric, F.Cu at (75.4, 72.6)
- added C43: 10uF, Capacitor_SMD:C_0805_2012Metric, F.Cu at (74.9, 75.2)
- added C44: 22uF, Capacitor_SMD:C_0603_1608Metric, F.Cu at (77.0, 83.2)
- added J7: 5V, Connector_PinHeader_2.54mm:PinHeader_1x02_P2.54mm_Vertical, F.Cu at (96.5, 72.3)
- added L1: 2.2µH, Inductor_SMD:L_Coilcraft_XxL4020, F.Cu at (77.7, 80.2)
- added U8: TPS62133, Package_DFN_QFN:VQFN-16-1EP_3x3mm_P0.5mm_EP1.68x1.68mm_ThermalVias, F.Cu at (78.0, 75.1)
- C10, C11, C12, C15, C16, C20, C21, C22, C23, C24, C25, C26, C27, C28, C29, C30, C31, C32, C33, C34, C35, C36, C37, C38, C39, C5, C6, C9: footprint Capacitor_SMD:C_0402_1005Metric -> Capacitor_SMD:C_0603_1608Metric
- J1: value PWR -> 3.3V
- moved C12 55.7 mm to (75.0, 123.9), turned to 180 degrees
- moved R12 54.8 mm to (72.1, 120.7)
- moved U6 54.8 mm to (76.5, 121.6)
- moved R11 54.8 mm to (72.1, 122.3)
- moved C11 54.1 mm to (79.1, 122.2)
- moved C1 9.74 mm to (71.8, 81.0), turned to 90 degrees
- moved C2 2.53 mm to (70.0, 81.0), turned to 90 degrees
- moved C30 2.04 mm to (79.7, 118.0)
- moved C24 1.99 mm to (88.1, 107.7)
- moved C23 1.55 mm to (86.6, 107.7)
- moved C35 1.49 mm to (79.7, 116.5)
- moved C20 1.34 mm to (79.7, 109.0)
- moved U1 1.19 mm to (70.3, 75.1), turned to 90 degrees
- moved C22 1.14 mm to (85.2, 107.7)
- moved C29 1.08 mm to (90.0, 115.8)
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Connections:
- C10 pad 1: +3.3V -> +5V
- C2 pad 2: Net-(JP1-B) -> +3.3V
- C5 pad 1: +3.3V -> +5V
- C6 pad 1: +3.3V -> +5V
- C9 pad 1: +3.3V -> +5V
- U1 pad 2: Net-(JP1-B) -> +3.3V
- U2 pad 3: +3.3V -> +5V
- U3 pad 3: +3.3V -> +5V
- U4 pad 3: +3.3V -> +5V
- U5 pad 3: +3.3V -> +5V
- USBC1 pad A4: +5V -> +12V
- USBC1 pad A9: +5V -> +12V
- USBC1 pad B4: +5V -> +12V
- USBC1 pad B9: +5V -> +12V
Routing:
- net /IMU_SDA: track 13.3 -> 76.8 mm, vias 0 -> 1
- net /IMU_SCL: track 17.9 -> 80.5 mm, vias 0 -> 1
- net +12V: track 0.00 -> 31.0 mm, vias 0 -> 3
- net +5V: track 64.5 -> 41.5 mm
- net GND: track 90.0 -> 112.9 mm, vias 44 -> 52
- net +3.3V: track 59.2 -> 72.4 mm, vias 33 -> 28
- net Net-(JP1-B): track 13.0 -> 0.00 mm
- net /AUDIO_SAI4_MCLK_B: track 37.4 -> 45.8 mm
- net /AUDIO_SAI4_SD_B: track 27.4 -> 35.0 mm
- net /AUDIO_DFSDM1_DATIN3: track 26.7 -> 33.1 mm
- net Net-(L1-Pad1): track 0.00 -> 5.63 mm
- net /FAN_SETUP: track 42.5 -> 37.6 mm
- net /JTDI: track 23.5 -> 27.9 mm
- net /FAN_ENABLE: track 22.0 -> 25.5 mm
- net /TRACESWO: track 30.1 -> 33.4 mm
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- added copper zone on In3.Cu, net +5V

Commit message: v3
Parts:
- C41: footprint Capacitor_SMD:C_0805_2012Metric -> Capacitor_SMD:C_0603_1608Metric
- SW1: value DFU -> BTN
- SW2: value RESET -> BTN
Changed lines of the file:
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@@
 		(4 "In1.Cu" power "GND1")
 		(6 "In2.Cu" signal "SIGNAL2")
-		(8 "In3.Cu" power "3.3V")
+		(8 "In3.Cu" power "PWR")
 		(10 "In4.Cu" power "GND2")
 		(2 "B.Cu" signal "SIGNAL3")
@@
 		)
 	)
-	(footprint "Capacitor_SMD:C_0805_2012Metric"
+	(footprint "Capacitor_SMD:C_0603_1608Metric"
 		(layer "F.Cu")
 		(at 105.15 73.39 90)
-		(descr "Capacitor SMD 0805 (2012 Metric), square (rectangular) end terminal, IPC-7351 nominal, (Body size source: IPC-SM-782 page 76, https://www.pcb-3d.com/wordpress/wp-content/uploads/ipc-sm-782a_amendment_1_and_2.pdf, https://docs.google.com/spreadsheets/d/1BsfQQcO9C6DZCsRaXUlFlo91Tg2WpOkGARC1WS5S8t0/edit?usp=sharing), generated with kicad-footprint-generator")
+		(descr "Capacitor SMD 0603 (1608 Metric), square (rectangular) end terminal, IPC-7351 nominal, (Body size source: IPC-SM-782 page 76, https://www.pcb-3d.com/wordpress/wp-content/uploads/ipc-sm-782a_amendment_1_and_2.pdf), generated with kicad-footprint-generator")
 		(tags "capacitor")
 		(property "Reference" "C41"
-			(at 2.13 -0.14 180)
+			(at 0 -1.43 90)
 			(layer "F.SilkS")
 			(effects
@@
 		)
 		(property "Value" "22uF"
-			(at 0 1.68 90)
+			(at 0 1.43 90)
 			(layer "F.Fab")
 			(effects
@@
 			)
 		)
-		(property "MPN" "CC0603MRX5R5BB226"
-			(at 0 0 90)
-			(unlocked yes)
-			(layer "F.Fab")
-			(hide yes)
-			(effects
-				(font
-					(size 1 1)
-					(thickness 0.15)
-				)
-			)
-		)
 		(property "Manufacturer" "YAGEO"
 			(at 0 0 90)
@@
 		(attr smd)
 		(fp_line
-			(start -0.261252 -0.735)
-			(end 0.261252 -0.735)
+			(start -0.14058 -0.51)
+			(end 0.14058 -0.51)
 			(stroke
 				(width 0.12)
@@
 		)
 		(fp_line
-			(start -0.261252 0.735)
-			(end 0.261252 0.735)
+			(start -0.14058 0.51)
+			(end 0.14058 0.51)
 			(stroke
 				(width 0.12)
@@
 		)
 		(fp_line
-			(start 1.7 -0.98)
-			(end 1.7 0.98)
+			(start 1.48 -0.73)
+			(end 1.48 0.73)
 			(stroke
 				(width 0.05)
@@
 		)
 		(fp_line
-			(start -1.7 -0.98)
-			(end 1.7 -0.98)
+			(start -1.48 -0.73)
+			(end 1.48 -0.73)
 			(stroke
 				(width 0.05)
@@
 		)
 		(fp_line
-			(start 1.7 0.98)
-			(end -1.7 0.98)
+			(start 1.48 0.73)
+			(end -1.48 0.73)
 			(stroke
 				(width 0.05)
@@
 		)
 		(fp_line
-			(start -1.7 0.98)
-			(end -1.7 -0.98)
+			(start -1.48 0.73)
+			(end -1.48 -0.73)
 			(stroke
 				(width 0.05)
@@
 		)
 		(fp_line
-			(start 1 -0.625)
-			(end 1 0.625)
+			(start 0.8 -0.4)
+			(end 0.8 0.4)
 			(stroke
 				(width 0.1)
@@
 		)
 		(fp_line
-			(start -1 -0.625)
-			(end 1 -0.625)
+			(start -0.8 -0.4)
+			(end 0.8 -0.4)
 			(stroke
 				(width 0.1)
@@
 		)
 		(fp_line
-			(start 1 0.625)
-			(end -1 0.625)
+			(start 0.8 0.4)
+			(end -0.8 0.4)
 			(stroke
 				(width 0.1)
@@
 		)
 		(fp_line
-			(start -1 0.625)
-			(end -1 -0.625)
+			(start -0.8 0.4)
+			(end -0.8 -0.4)
 			(stroke
 				(width 0.1)
@@
 			(effects
 				(font
-					(size 0.5 0.5)
-					(thickness 0.08)
+					(size 0.4 0.4)
+					(thickness 0.06)
 				)
 			)
 		)
 		(pad "1" smd roundrect
-			(at -0.95 0 90)
-			(size 1 1.45)
+			(at -0.775 0 90)
+			(size 0.9 0.95)
 			(layers "F.Cu" "F.Mask" "F.Paste")
 			(roundrect_rratio 0.25)
@@
 		)
 		(pad "2" smd roundrect
-			(at 0.95 0 90)
-			(size 1 1.45)
+			(at 0.775 0 90)
+			(size 0.9 0.95)
 			(layers "F.Cu" "F.Mask" "F.Paste")
 			(roundrect_rratio 0.25)
@@
 		)
 		(embedded_fonts no)
-		(model "${KICAD9_3DMODEL_DIR}/Capacitor_SMD.3dshapes/C_0805_2012Metric.step"
+		(model "${KICAD9_3DMODEL_DIR}/Capacitor_SMD.3dshapes/C_0603_1608Metric.step"
 			(offset
 				(xyz 0 0 0)
@@
 			)
 		)
-		(property "Value" "DFU"
+		(property "Value" "BTN"
 			(at 0 3 90)
 			(layer "F.Fab")
@@
 			)
 		)
-		(property "Value" "RESET"
+		(property "Value" "BTN"
 			(at 0 3 90)
 			(layer "F.Fab")
