File: hw/Asius2/Asius2.kicad_sch (KiCad schematic)
At the start: 77 parts, among them J1 PWR, J2 Hat, J3 Others, J4 Fan, J5 Audio, J6 SWD, SW1 DFU, SW2 RESET, U1 AMS1117-3.3, U2 TJA1042T, U3 TJA1042T, U4 TJA1042T, U5 TJA1042T, U6 LSM6DSOXTR, U7 STM32H725AGIx, Y1 Crystal_GND24

Commit message: v2
Parts:
- removed JP1: ~, Jumper:SolderJumper-2_P1.3mm_Bridged_RoundedPad1.0x1.5mm, symbol Jumper:SolderJumper_2_Bridged
- added C42: 3.3nF, Capacitor_SMD:C_0603_1608Metric, symbol Device:C_Small
- added C43: 10uF, Capacitor_SMD:C_0805_2012Metric, symbol Device:C_Small
- added C44: 22uF, Capacitor_SMD:C_0603_1608Metric, symbol Device:C_Small
- added J7: 5V, Connector_PinHeader_2.54mm:PinHeader_1x02_P2.54mm_Vertical, symbol Connector:Conn_01x02_Pin
- added L1: 2.2µH, Inductor_SMD:L_Coilcraft_XxL4020, symbol Device:L
- added U8: TPS62133, Package_DFN_QFN:VQFN-16-1EP_3x3mm_P0.5mm_EP1.68x1.68mm_ThermalVias, symbol Regulator_Switching:TPS62133
- C1: JLCPCB Part # (none) -> C106245; MFR.Part # (none) -> CC0603JRNPO9BN100; MPN CC0603JRNPO9BN100 -> (none)
- C10, C11, C12, C15, C16, C20, C21, C22, C23, C24, C25, C26, C27, C28, C29, C30, C31, C32, C33, C34, C35, C36, C37, C38, C39, C5, C6, C9: footprint Capacitor_SMD:C_0402_1005Metric -> Capacitor_SMD:C_0603_1608Metric; JLCPCB Part # (none) -> C14663; MFR.Part # (none) -> CC0603KRX7R9BB104; MPN CC0402KRX7R7BB104 -> (none)
- C13, C14: JLCPCB Part # (none) -> C107037; MFR.Part # (none) -> CC0603JRNPO9BN150; MPN CC0603JRNPO9BN150 -> (none)
- C17, C18, C19: JLCPCB Part # (none) -> C106213; MFR.Part # (none) -> CC0603KRX5R6BB225; MPN CC0603KRX5R5BB225 -> (none)
- C2: JLCPCB Part # (none) -> C105620; MFR.Part # (none) -> CC0603JRNPO9BN220; MPN CC0603JRNPO9BN220 -> (none)
- C3, C4, C7, C8: JLCPCB Part # (none) -> C106217; MFR.Part # (none) -> CC0603KRX7R8BB223; MPN CC0603KRX7R8BB223 -> (none)
- C40: JLCPCB Part # (none) -> C3345; MFR.Part # (none) -> RVT1A221M0605; MPN RVT1A221M0605 -> (none)
- C41: JLCPCB Part # (none) -> C109448; MFR.Part # (none) -> CC0603MRX5R5BB226; MPN CC0603MRX5R5BB226 -> (none)
- D1: JLCPCB Part # (none) -> C3029073; MFR.Part # (none) -> SZYY1209RGB-B 4pin; MPN SZYY1209RGB-B 4pin -> (none)
- J1: value PWR -> 3.3V; MFR.Part # (none) -> -; MPN - -> (none)
- J2: MFR.Part # (none) -> -; MPN DS1023-2*20SF11 -> (none); Manufacturer CONNFLY Elec -> -; now left out of the parts list
- J3, J4, J5, J6: MFR.Part # (none) -> -; MPN - -> (none)
- R1, R2: JLCPCB Part # (none) -> C122969; MFR.Part # (none) -> RT0603BRD075K1L; MPN RT0603BRD075K1L -> (none)
- R10, R3, R4, R5, R6, R7, R8, R9: JLCPCB Part # (none) -> C245989; MFR.Part # (none) -> RC0603FR-0762RL; MPN RC0603FR-0762RL -> (none)
- R11, R12, R16, R17: JLCPCB Part # (none) -> C98220; MFR.Part # (none) -> RC0603FR-0710KL; MPN RC0603FR-0710KL -> (none)
- R13: JLCPCB Part # (none) -> C105881; MFR.Part # (none) -> RC0603FR-07330RL; MPN RC0603FR-07330RL -> (none)
- R14, R15: JLCPCB Part # (none) -> C105588; MFR.Part # (none) -> RC0603FR-07100RL; MPN RC0603FR-07100RL -> (none)
- SW1: JLCPCB Part # (none) -> C79161; MFR.Part # (none) -> EVQP2R02M; MPN EVQP2R02M -> (none)
- SW2: JLCPCB Part # (none) -> C79161; MFR.Part # (none) -> EVQP2R02M; MPN EVQP2R02M -> (none); Manufacturer PANASONIC -> Panasonic
- U1: JLCPCB Part # (none) -> C6186; MFR.Part # (none) -> AMS1117-3.3; MPN AMS1117-3.3 -> (none)
- U2, U3, U4, U5: JLCPCB Part # (none) -> C53670; MFR.Part # (none) -> TJA1042T/1J; MPN TJA1042T/1J -> (none)
- U6: JLCPCB Part # (none) -> C481766; MFR.Part # (none) -> LSM6DSOXTR; MPN LSM6DSOXTR -> (none)
- U7: JLCPCB Part # (none) -> C730148; MFR.Part # (none) -> STM32H725AGI6; MPN STM32H725AGI6 -> (none)
- USBC1: JLCPCB Part # (none) -> C129018; MFR.Part # (none) -> TYPE-C-31-M-04; MPN TYPE-C-31-M-04 -> (none)
- Y1: JLCPCB Part # (none) -> C9006; MFR.Part # (none) -> X322525MOB4SI; MPN X322525MOB4SI -> (none)
Connections:
- net +3.3V: now also C2.2, U1.2 (VO); no longer C10.1, C5.1, C6.1, C9.1, U2.3 (VCC), U3.3 (VCC), U4.3 (VCC), U5.3 (VCC)
- net +5V: now also C10.1, C5.1, C6.1, C9.1, U2.3 (VCC), U3.3 (VCC), U4.3 (VCC), U5.3 (VCC), C44.2, J7.2 (Pin_2), L1.2, U8.14 (VOS); no longer USBC1.A4 (VBUS), USBC1.A9 (VBUS), USBC1.B4 (VBUS), USBC1.B9 (VBUS)
- net GND: now also C42.1, C43.1, C44.1, J7.1 (Pin_1), U8.15 (GND), U8.16 (GND), U8.17 (GND), U8.5 (FB), U8.6 (GND), U8.7 (FSW), U8.8 (DEF)
- new net: L1.1, U8.1 (SW), U8.2 (SW), U8.3 (SW)
- new net: C42.2, U8.9 (SS/TR)
- new net +12V: C43.2, U8.10 (VIN), U8.11 (VIN), U8.12 (VIN), U8.13 (EN), USBC1.A4 (VBUS), USBC1.A9 (VBUS), USBC1.B4 (VBUS), USBC1.B9 (VBUS)
- no-connect marks 107 -> 108
Other:
- moved on the sheet: C1, C2, U1

Commit message: v3
Parts:
- C41: footprint Capacitor_SMD:C_0805_2012Metric -> Capacitor_SMD:C_0603_1608Metric
- SW1: value DFU -> BTN
- SW2: value RESET -> BTN
